Commit message: [add] connect to true so100

File: resources/SO_5DOF_ARM100_8j_URDF.SLDASM copy.urdf (robot description, URDF)
Before this commit: robot SO_5DOF_ARM100_8j_URDF.SLDASM, 6 links, 5 joints
Links:
- added link Moving Jaw, mass 0.0202443794940372; collision mesh filename=package://SO_5DOF_ARM100_8j_URDF.SLDASM/meshes/Moving Jaw.S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; visual mesh filename=package://SO_5DOF_ARM100_8j_URDF.SLDASM/meshes/Moving Jaw.S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
Joints:
- added joint Jaw: type continuous, parent Fixed_Jaw, child Moving Jaw, origin xyz=-0.0202 -0.0244 0 rpy=3.1416 0 3.1416, axis 0 0 1

File: resources/so100_tcp.urdf (robot description, URDF)
Before this commit: robot SO_5DOF_ARM100_8j_URDF.SLDASM, 6 links, 5 joints
Links:
- added link tcp, mass 0.0929859131176897; collision mesh filename=package://SO_5DOF_ARM100_8j_URDF.SLDASM/meshes/Fixed_Jaw.STL; visual mesh filename=package://SO_5DOF_ARM100_8j_URDF.SLDASM/meshes/Fixed_Jaw.STL
Joints:
- added joint j_tcp: type fixed, parent Fixed_Jaw, child tcp, origin xyz=0 -0.1 0 rpy=0 0 0, axis 0 1 0
