Commit message: [add] add joints limits in urdf

File: resources/urdf/so100_tcp copy.urdf (robot description, URDF)
Before this commit: robot SO_5DOF_ARM100_8j_URDF.SLDASM, 7 links, 6 joints
Joints:
- joint Elbow: limit lower=-1.78 upper=1.57 effort=10.0 velocity=1.0 -> (none); type revolute -> continuous
- joint Pitch: limit lower=-1.8 upper=1.9 effort=10.0 velocity=1.0 -> (none); type revolute -> continuous
- joint Rotation: limit lower=-1.76 upper=1.8 effort=10.0 velocity=1.0 -> (none); type revolute -> continuous
- joint Wrist_Pitch: limit lower=-3.566 upper=0.19 effort=10.0 velocity=1.0 -> (none); type revolute -> continuous
- joint Wrist_Roll: limit lower=-1.73 upper=1.71 effort=10.0 velocity=1.0 -> (none); type revolute -> continuous
- joint j_tcp: limit lower=-0.15 upper=1.96 effort=10.0 velocity=1.0 -> (none)
